Commit message: Add the camera simulation.
Signed-off-by: Jean-Christophe PINCE <jcpince@gmail.com>

File: bobby_description/urdf/bobby.xacro (robot description, xacro)
@@ -59,4 +59,29 @@
         </inertial>
     </link>
+    <joint name="camera_joint" type="fixed">
+        <origin xyz="${-cameraSize+chassisLength/2} 0 ${cameraSize+wheelRadius+cameraSize/2}" rpy="0 0 0"/>
+        <parent link="chassis"/>
+        <child link="camera"/>
+    </joint>
+    <link name="camera">
+        <collision>
+            <origin xyz="0 0 0" rpy="0 0 0"/>
+            <geometry>
+                <box size="${cameraSize} ${cameraSize} ${cameraSize}"/>
+            </geometry>
+        </collision>
+        <visual>
+            <origin xyz="0 0 0" rpy="0 0 0"/>
+            <geometry>
+                <box size="${cameraSize} ${cameraSize} ${cameraSize}"/>
+            </geometry>
+            <material name="blue"/>
+        </visual>
+        <inertial>
+            <mass value="${cameraMass}" />
+            <origin xyz="0 0 0" rpy="0 0 0"/>
+            <box_inertia m="${cameraMass}" x="${cameraSize}" y="${cameraSize}" z="${cameraSize}" />
+        </inertial>
+    </link>
     <wheel lr="left" tY="1"/>
     <wheel lr="right" tY="-1"/>

Commit message: Add hokuyo laser.
Signed-off-by: Jean-Christophe PINCE <jcpince@gmail.com>

File: bobby_description/urdf/bobby.xacro (robot description, xacro)
@@ -84,4 +84,30 @@
         </inertial>
     </link>
+    <joint name="hokuyo_joint" type="fixed">
+        <axis xyz="0 1 0" />
+        <origin xyz="${-cameraSize+chassisLength/2} ${cameraSize} ${cameraSize+wheelRadius+cameraSize/2}" rpy="0 0 0"/>
+        <parent link="chassis"/>
+        <child link="hokuyo_link"/>
+    </joint>
+    <!-- Hokuyo Laser -->
+    <link name="hokuyo_link">
+        <collision>
+            <origin xyz="0 0 0" rpy="0 0 0"/>
+            <geometry>
+                <box size="0.1 0.1 0.1"/>
+            </geometry>
+        </collision>
+        <visual>
+            <origin xyz="0 0 0" rpy="0 0 0"/>
+            <geometry>
+                <box size="${cameraSize} ${cameraSize} ${cameraSize}"/>
+            </geometry>
+        </visual>
+        <inertial>
+            <mass value="1e-5" />
+            <origin xyz="0 0 0" rpy="0 0 0"/>
+            <inertia ixx="1e-6" ixy="0" ixz="0" iyy="1e-6" iyz="0" izz="1e-6" />
+        </inertial>
+    </link>
     <wheel lr="left" tY="1"/>
     <wheel lr="right" tY="-1"/>
